File: eagle/h2oiq/h2oiq_v4.brd (EAGLE design)
At the start: 40.6 x 43.2 mm, 23 parts, among them IC1 MEGA88, T2 BC846, U1 MAX1704X

Commit message: minor pcb change
Routing:
- net VCC: track 68.1 -> 66.1 mm
- net N$10: track 17.4 -> 18.2 mm, vias 3 -> 2
Other:
- board text added: "LiPo 100mAh Batt"
Changed lines of the file:
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@@
 <wire x1="13.335" y1="26.035" x2="0.635" y2="26.035" width="0.3048" layer="21"/>
 <wire x1="0.635" y1="26.035" x2="0.635" y2="0.635" width="0.3048" layer="21"/>
+<text x="6.985" y="3.175" size="1.27" layer="21" align="center">LiPo 100mAh
+Batt</text>
 </plain>
 <attributes>
@@
 <wire x1="14.478" y1="13.97" x2="14.4" y2="13.82" width="0.254" layer="16"/>
 <via x="30.734" y="24.638" extent="1-16" drill="0.6096"/>
-<wire x1="18.288" y1="23.368" x2="23.876" y2="23.368" width="0.254" layer="16"/>
 <wire x1="15.494" y1="20.574" x2="18.288" y2="23.368" width="0.254" layer="16"/>
 <wire x1="15.494" y1="13.97" x2="15.494" y2="20.574" width="0.254" layer="16"/>
@@
 <wire x1="30.226" y1="25.4" x2="30.734" y2="24.638" width="0.254" layer="16"/>
 <wire x1="24.638" y1="25.4" x2="30.226" y2="25.4" width="0.254" layer="16"/>
-<wire x1="23.876" y1="23.368" x2="24.638" y2="25.4" width="0.254" layer="16"/>
 <wire x1="24.32" y1="26.65" x2="22.665" y2="26.65" width="0.3048" layer="1"/>
 <wire x1="22.665" y1="26.65" x2="22.225" y2="27.09" width="0.3048" layer="1"/>
@@
 <wire x1="31.75" y1="26.67" x2="35.55" y2="26.67" width="0.3048" layer="16"/>
 <wire x1="35.55" y1="26.67" x2="36.4" y2="25.82" width="0.3048" layer="16"/>
+<wire x1="18.288" y1="23.368" x2="20.828" y2="23.368" width="0.3048" layer="16"/>
+<wire x1="20.828" y1="23.368" x2="23.114" y2="25.654" width="0.3048" layer="16"/>
 </signal>
 <signal name="N$2">
@@
 <contactref element="IC1" pad="1"/>
 <wire x1="29.02" y1="23.65" x2="32.54" y2="23.65" width="0.3048" layer="1"/>
+<wire x1="33.02" y1="10.66" x2="33.02" y2="12.7" width="0.3048" layer="1"/>
+<via x="33.02" y="12.7" extent="1-16" drill="0.6"/>
 <wire x1="32.54" y1="23.65" x2="33.02" y2="24.13" width="0.3048" layer="1"/>
 <via x="33.02" y="24.13" extent="1-16" drill="0.6"/>
-<via x="32.54" y="23.65" extent="1-16" drill="0.6"/>
-<wire x1="32.54" y1="23.65" x2="32.54" y2="13.18" width="0.3048" layer="16"/>
-<wire x1="32.54" y1="13.18" x2="33.02" y2="12.7" width="0.3048" layer="16"/>
-<via x="33.02" y="12.7" extent="1-16" drill="0.6"/>
-<wire x1="33.02" y1="10.66" x2="33.02" y2="12.7" width="0.3048" layer="1"/>
+<wire x1="33.02" y1="24.13" x2="33.02" y2="23.495" width="0.3048" layer="16"/>
+<wire x1="33.02" y1="23.495" x2="32.385" y2="22.86" width="0.3048" layer="16"/>
+<wire x1="32.385" y1="22.86" x2="32.385" y2="13.335" width="0.3048" layer="16"/>
+<wire x1="32.385" y1="13.335" x2="33.02" y2="12.7" width="0.3048" layer="16"/>
 </signal>
 <signal name="N$26">
@@
 </board>
 </drawing>
+<compatibility>
+<note version="6.3" minversion="6.2.2" severity="warning">
+Since Version 6.2.2 text objects can contain more than one line,
+which will not be processed correctly with this version.
+</note>
+</compatibility>
 </eagle>

Commit message: New board adjustments
Parts:
- BATTCON: value (none) -> 3.3V
- C1, C2, C5: device SparkFun:0402-CAP -> rcl:C0603K
- R2: device rcl:R0603 -> resistor:R0603
- U$1, U$3, U$4, U$5: device SparkFun:BUTTON-CONDUCTIVE -> SparkFun:TACTILE_SWITCH_SMD
- moved U$1 1.27 mm to (20.3, 12.7)
- moved U$3 1.27 mm to (27.9, 12.7), turned to 270 degrees
- moved LED1 1.27 mm to (33.0, 8.89)
- moved R4 1.27 mm to (33.0, 5.08)
- moved R2 0.64 mm to (21.6, 27.9)
- moved LIPOREG 0.63 mm to (8.26, 21.6)
- turned U$4 to 270 degrees
Connections:
- net N$1 renamed VIN
Routing:
- net GND: track 39.2 -> 42.4 mm
- net N$20: track 22.6 -> 19.8 mm
- net N$10: track 18.2 -> 19.5 mm
- net N$16: track 12.8 -> 11.8 mm
- net N$18: track 13.6 -> 14.4 mm
- net VCC: track 66.1 -> 66.9 mm
- net N$3: track 27.4 -> 26.6 mm
- net N$12: track 19.9 -> 20.6 mm
- net VIN: track 10.0 -> 9.42 mm
