File: eagle/h2oiq/h2oiq_v4.sch (EAGLE design)
At the start: 23 parts, among them IC1 MEGA88, T2 BC846, U1 MAX1704X

Commit message: New board adjustments
Parts:
- BATTCON: value (none) -> 3.3V
- C1, C2, C5: device SparkFun:CAP0402-CAP -> rcl:C-USC0603K
- R2: device rcl:R-US_R0603 -> resistor:R-US_R0603
- U$1, U$3, U$4, U$5: device SparkFun:BUTTON-CONDUCTIVESMD -> SparkFun:TAC_SWITCHSMD
Connections:
- net N$1 renamed VIN
Other:
- moved on the sheet: C1, C2, C5
